File: _autosave-Interface_PCB.kicad_sch (KiCad schematic)
At the start: 25 parts, among them IC1 STM32L412RBT6P, J1 USB_B, J2 AVR-JTAG-10, J3 Conn_01x04, J4 Conn_01x04, J5 Conn_01x04, J6 Conn_01x04, U1 AMS1117, Y1 Crystal, Y2 Crystal

Commit message: Full Schematic Rev 1.0
Parts:
- removed C? (x2): C, symbol Device:C
- removed NT?: NetTie_3_Tee, symbol Device:NetTie_3_Tee
- removed R? (x2): R, symbol Device:R
- removed U1, U?: AMS1117, Package_TO_SOT_SMD:SOT-223-3_TabPin2, symbol Regulator_Linear:AMS1117
- added C? (x5): 100n, symbol Device:C
- added C? (x3): 22uF, symbol Device:C
- added C? (x5): 4.7u, symbol Device:C
- added C?: 1u, symbol Device:C
- added C? (x2): 10n, symbol Device:C
- added L?: 39nH, symbol Device:L
- added NT?: NetTie_3_Tee, symbol Device:NetTie_3_Tee
- added U?: AMS1117-3.3, Package_TO_SOT_SMD:SOT-223-3_TabPin2, symbol Regulator_Linear:AMS1117-3.3
Connections:
- net +3V3: now also C?.1, C?.1, C?.1, C?.1, C?.1, C?.1, C?.1, C?.1, C?.1, C?.1, C?.1, C?.1, L?.1
- net GND: now also IC1.12 (VSSA/VREF-), C?.2, C?.2, C?.2, C?.2, C?.2, C?.2, C?.2, C?.2, C?.2, C?.2, C?.2, C?.2, C?.2, U?.1 (GND)
- net VBUS: now also NT?.1
- net VEXT: now also C?.1, NT?.2
- net +3.3VA: now reaches IC1.13 (VDDA/VREF+)
- net +3.3VA: now also C?.1, L?.2
- new net: C?.1, U?.2 (VO)
- new net: C?.1, NT?.3, U?.3 (VI)
- new net: C?.2, C?.2, C?.2
Other:
- note added: "?? check if reverse polarity protection is needed ??"
- note added: "Analog Power filter network. kept extra capacitor pad if required. filtering with a 39nH inductor."
- note added: "Fixed output LDO for 3.3 V rail. Input is through USB or external Power Pin. Probably should add footprint for either ferrite or inductor between VEXT and nettie."
- note added: "The 4.7uF capacitor is the Bulk decoupling capacitor. Place it close to the VDD VSS pins. The rest of the decoupling is through the other caps and pwr and gnd planes."
- moved on the sheet: Cl1, Cl2, Cl3, Cl4, D1, D2, J1, J2, J3, J4, J5, J6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
